File: clock/clock.kicad_sch (KiCad schematic)
At the start: 43 parts, among them J1 Conn_01x06, J2 Power_inlet_vertical, J3 Conn_02x03_Odd_Even, J4 Conn_01x05, J5 Conn_01x05, SW1 Omron_B3F_SPST, SW2 Omron_B3F_SPST, SW3 Omron_B3F_SPST, SW4 Omron_B3F_SPST, U1 ATmega328-PU, U2 L7805, U3 MAX7219, U4 DS1307_DIP-8, Y1 Crystal_16MHz, Y2 Crystal_32768Hz

Commit message: pretty close to done
Connections:
- net BTH_DWN is gone; now on net BTN_DWN: U1.4 (PD2)
Changed lines of the file:
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@@
     )
   )
-  (global_label "BTH_DWN" (shape input) (at 54.61 97.79 0) (fields_autoplaced)
+  (global_label "BTN_DWN" (shape input) (at 54.61 97.79 0) (fields_autoplaced)
     (effects (font (size 1.27 1.27)) (justify left))
     (property "Intersheet References" "${INTERSHEET_REFS}" (id 0) (at 65.6107 97.7106 0)

Commit message: 70% there
Connections:
- net DEBUG_4: now also J4.1 (Pin_1); no longer J4.2 (Pin_2)
- net DEBUG_5: now also J4.2 (Pin_2); no longer J4.3 (Pin_3)
- net DEBUG_6: now also J4.3 (Pin_3); no longer J4.4 (Pin_4)
- net VCC: now also J4.4 (Pin_4); no longer J4.1 (Pin_1)
Changed lines of the file:
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@@
     (stroke (width 0) (type default) (color 0 0 0 0))
   )
+  (wire (pts (xy 28.575 139.7) (xy 31.75 139.7))
+    (stroke (width 0) (type default) (color 0 0 0 0))
+  )
   (wire (pts (xy 39.37 41.91) (xy 39.37 40.64))
     (stroke (width 0) (type default) (color 0 0 0 0))
@@
     (stroke (width 0) (type default) (color 0 0 0 0))
   )
-  (wire (pts (xy 28.575 144.78) (xy 31.75 144.78))
-    (stroke (width 0) (type default) (color 0 0 0 0))
-  )
   (wire (pts (xy 208.28 128.27) (xy 205.74 128.27))
     (stroke (width 0) (type default) (color 0 0 0 0))
@@
     (stroke (width 0) (type default) (color 0 0 0 0))
   )
+  (wire (pts (xy 26.035 144.78) (xy 26.035 147.955))
+    (stroke (width 0) (type default) (color 0 0 0 0))
+  )
   (polyline (pts (xy 283.21 106.045) (xy 283.21 149.86))
     (stroke (width 0) (type default) (color 0 0 0 0))
@@
     (stroke (width 0) (type default) (color 0 0 0 0))
   )
-  (wire (pts (xy 28.575 142.24) (xy 31.75 142.24))
-    (stroke (width 0) (type default) (color 0 0 0 0))
-  )
   (wire (pts (xy 142.875 157.48) (xy 142.875 167.005))
     (stroke (width 0) (type default) (color 0 0 0 0))
@@
     (stroke (width 0) (type default) (color 0 0 0 0))
   )
+  (wire (pts (xy 28.575 137.16) (xy 31.75 137.16))
+    (stroke (width 0) (type default) (color 0 0 0 0))
+  )
   (wire (pts (xy 52.07 59.69) (xy 55.245 59.69))
     (stroke (width 0) (type default) (color 0 0 0 0))
@@
     (stroke (width 0) (type default) (color 0 0 0 0))
   )
-  (wire (pts (xy 30.48 137.16) (xy 31.75 137.16))
-    (stroke (width 0) (type default) (color 0 0 0 0))
-  )
   (polyline (pts (xy 106.68 88.9) (xy 106.68 120.65))
     (stroke (width 0) (type default) (color 0 0 0 0))
@@
     (stroke (width 0) (type default) (color 0 0 0 0))
   )
+  (wire (pts (xy 31.75 144.78) (xy 26.035 144.78))
+    (stroke (width 0) (type default) (color 0 0 0 0))
+  )
   (wire (pts (xy 220.98 62.865) (xy 233.68 62.865))
     (stroke (width 0) (type default) (color 0 0 0 0))
@@
     (stroke (width 0) (type default) (color 0 0 0 0))
   )
-  (wire (pts (xy 30.48 136.525) (xy 30.48 137.16))
-    (stroke (width 0) (type default) (color 0 0 0 0))
-  )
   (wire (pts (xy 124.46 184.785) (xy 129.54 184.785))
     (stroke (width 0) (type default) (color 0 0 0 0))
@@
     (stroke (width 0) (type default) (color 0 0 0 0))
   )
+  (wire (pts (xy 28.575 142.24) (xy 31.75 142.24))
+    (stroke (width 0) (type default) (color 0 0 0 0))
+  )
   (wire (pts (xy 133.35 20.32) (xy 143.51 20.32))
     (stroke (width 0) (type default) (color 0 0 0 0))
@@
     (stroke (width 0) (type default) (color 0 0 0 0))
   )
-  (wire (pts (xy 28.575 139.7) (xy 31.75 139.7))
-    (stroke (width 0) (type default) (color 0 0 0 0))
-  )
   (wire (pts (xy 86.36 72.39) (xy 91.44 72.39))
     (stroke (width 0) (type default) (color 0 0 0 0))
@@
     )
   )
-  (global_label "DEBUG_4" (shape input) (at 28.575 139.7 180) (fields_autoplaced)
+  (global_label "DEBUG_4" (shape input) (at 28.575 137.16 180) (fields_autoplaced)
     (effects (font (size 1.27 1.27)) (justify right))
-    (property "Intersheet References" "${INTERSHEET_REFS}" (id 0) (at 17.6952 139.6206 0)
+    (property "Intersheet References" "${INTERSHEET_REFS}" (id 0) (at 17.6952 137.0806 0)
       (effects (font (size 1.27 1.27)) (justify right) hide)
     )
@@
     )
   )
-  (global_label "DEBUG_6" (shape input) (at 28.575 144.78 180) (fields_autoplaced)
+  (global_label "DEBUG_6" (shape input) (at 28.575 142.24 180) (fields_autoplaced)
     (effects (font (size 1.27 1.27)) (justify right))
-    (property "Intersheet References" "${INTERSHEET_REFS}" (id 0) (at 17.6952 144.7006 0)
+    (property "Intersheet References" "${INTERSHEET_REFS}" (id 0) (at 17.6952 142.1606 0)
       (effects (font (size 1.27 1.27)) (justify right) hide)
     )
@@
     )
   )
-  (global_label "DEBUG_5" (shape input) (at 28.575 142.24 180) (fields_autoplaced)
+  (global_label "DEBUG_5" (shape input) (at 28.575 139.7 180) (fields_autoplaced)
     (effects (font (size 1.27 1.27)) (justify right))
-    (property "Intersheet References" "${INTERSHEET_REFS}" (id 0) (at 17.6952 142.1606 0)
+    (property "Intersheet References" "${INTERSHEET_REFS}" (id 0) (at 17.6952 139.6206 0)
       (effects (font (size 1.27 1.27)) (justify right) hide)
     )
@@
     (pin "8")
   )
-  (symbol (lib_id "HPS:VCC") (at 30.48 136.525 0) (unit 1)
-    (in_bom yes) (on_board yes)
-    (property "Reference" "#PWR030" (id 0) (at 30.48 140.335 0)
-      (effects (font (size 1.27 1.27)) hide)
-    )
-    (property "Value" "VCC" (id 1) (at 30.48 132.715 0))
-    (property "Footprint" "" (id 2) (at 30.48 136.525 0)
-      (effects (font (size 1.27 1.27)) hide)
-    )
-    (property "Datasheet" "" (id 3) (at 30.48 136.525 0)
-      (effects (font (size 1.27 1.27)) hide)
-    )
-    (pin "1")
-  )
   (symbol (lib_id "HPS:C_0805_0.1uf") (at 26.67 35.56 90) (unit 1)
     (in_bom yes) (on_board yes)
@@
     (pin "1")
   )
+  (symbol (lib_id "HPS:VCC") (at 26.035 147.955 180) (unit 1)
+    (in_bom yes) (on_board yes)
+    (property "Reference" "#PWR?" (id 0) (at 26.035 144.145 0)
+      (effects (font (size 1.27 1.27)) hide)
+    )
+    (property "Value" "VCC" (id 1) (at 26.035 151.765 0))
+    (property "Footprint" "" (id 2) (at 26.035 147.955 0)
+      (effects (font (size 1.27 1.27)) hide)
+    )
+    (property "Datasheet" "" (id 3) (at 26.035 147.955 0)
+      (effects (font (size 1.27 1.27)) hide)
+    )
+    (pin "1")
+  )
   (symbol (lib_id "HPS:GND") (at 130.175 114.3 0) (unit 1)
     (in_bom yes) (on_board yes) (fields_autoplaced)
@@
       (reference "#PWR029") (unit 1) (value "GND") (footprint "")
     )
-    (path "/4333a74f-9f73-4c95-ae69-208dd95f958b"
-      (reference "#PWR030") (unit 1) (value "VCC") (footprint "")
-    )
     (path "/0ef66e02-311b-456b-bd24-c5125a12c1f6"
       (reference "#PWR031") (unit 1) (value "GND") (footprint "")
@@
       (reference "#PWR0102") (unit 1) (value "GND") (footprint "")
     )
+    (path "/c2f0bede-7012-425b-af8e-1abede33b62c"
+      (reference "#PWR?") (unit 1) (value "VCC") (footprint "")
+    )
     (path "/8c33e279-28d8-480f-bd32-b858d3bc749f"
