File: clock/clock.kicad_pcb (KiCad board)
At the start: 2 copper layers, 140 x 90 mm, 4 parts

Commit message: lil changes
Parts:
- added BT1: Battery_Cell, footprints:BatteryHolder_Keystone_106_1x20mm, F.Cu at (110.7, 121.9)
- added C1: C_0805_0.1uf, footprints:C_0805_2012Metric, F.Cu at (302.6, 85.8)
- added C2: C_0805_0.1uf, footprints:C_0805_2012Metric, F.Cu at (313.8, 80.9)
- added C3: C_0805_22pf, footprints:C_0805_2012Metric, F.Cu at (267.9, 123.6)
- added C4: C_0805_22pf, footprints:C_0805_2012Metric, F.Cu at (245.4, 127.5)
- added C5: C_0805_0.1uf, footprints:C_0805_2012Metric, F.Cu at (245.4, 121.6)
- added C6: C_0805_1uf, footprints:C_0805_2012Metric, F.Cu at (302.6, 91.7)
- added C7: C_0805_0.1uf, footprints:C_0805_2012Metric, F.Cu at (254.3, 125.7)
- added C8: C_0805_1uf, footprints:C_0805_2012Metric, F.Cu at (284.8, 106.4)
- added C9: C_0805_0.1uf, footprints:C_0805_2012Metric, F.Cu at (325.9, 69.9)
- added D1: LED_0805, footprints:LED_0805_2012Metric, F.Cu at (256.7, 110.5)
- added DS1: LED_Display_1001, footprints:Adafruit-1001-0-0-MFG, F.Cu at (149.9, 86.4)
- added J1: Conn_01x06, footprints:PinHeader_1x06_P2.54mm_Vertical, F.Cu at (252.1, 107.9)
- added J2: PJ-102AH, footprints:PJ-102AH, F.Cu at (266.6, 111.3)
- added J3: Conn_02x03_Odd_Even, footprints:PinHeader_2x03_P2.54mm_Vertical, F.Cu at (274.1, 108.2)
- added R1: R_0805_10K, footprints:R_0805_2012Metric, F.Cu at (256.6, 113.5)
- added R10: R_0805_10K, footprints:R_0805_2012Metric, F.Cu at (249.9, 124.4)
- added R11: R_0805_10K, footprints:R_0805_2012Metric, F.Cu at (313.8, 78.0)
- added R12: R_0805_10K, footprints:R_0805_2012Metric, F.Cu at (296.0, 95.6)
- added R2: R_0805_47, footprints:R_0805_2012Metric, F.Cu at (258.7, 125.7)
- added R3: R_0805_47, footprints:R_0805_2012Metric, F.Cu at (307.0, 85.8)
- added R4: R_0805_2.2K, footprints:R_0805_2012Metric, F.Cu at (249.9, 127.4)
- added R5: R_0805_4.7K, footprints:R_0805_2012Metric, F.Cu at (302.6, 88.8)
- added R6: R_0805_4.7K, footprints:R_0805_2012Metric, F.Cu at (263.1, 125.7)
- added R7: R_0805_22K, footprints:R_0805_2012Metric, F.Cu at (284.8, 103.5)
- added R8: PhotoconductivePhotocell, footprints:R_LDR_4.9x4.2mm_P2.54mm_Vertical, F.Cu at (267.6, 119.2)
- added R9: R_0805_100K, footprints:R_0805_2012Metric, F.Cu at (245.4, 124.5)
- added SW1: Omron_B3F_SPST, footprints:SW_SPST_Omron_B3FS-100xP, F.Cu at (318.2, 72.4)
- added SW2: Omron_B3F_SPST, footprints:SW_SPST_Omron_B3FS-100xP, F.Cu at (306.0, 80.4)
- added SW3: Omron_B3F_SPST, footprints:SW_SPST_Omron_B3FS-100xP, F.Cu at (288.3, 98.1)
- added SW4: Omron_B3F_SPST, footprints:SW_SPST_Omron_B3FS-100xP, F.Cu at (260.1, 120.3)
- added U1: ATmega328-PU, footprints:DIP-28_W7.62mm, F.Cu at (120.6, 110.5)
- added U2: L7805, footprints:TO-252-2, F.Cu at (306.4, 72.5)
- added U3: MAX7219, footprints:DIP-24_W7.62mm, F.Cu at (156.2, 100.3)
- added U4: DS1307_DIP-8, footprints:DIP-8_W7.62mm, F.Cu at (133.3, 123.2)
- added Y1: Crystal_16MHz, footprints:Crystal_SMD_HC49-SD, F.Cu at (235.9, 123.2)
- added Y2: Crystal_32768Hz, footprints:Crystal_SMD_2Pin_3.2x1.5mm, F.Cu at (257.0, 107.3)
