File: clock/clock.kicad_pcb (KiCad board)
At the start: 2 copper layers, 140 x 90 mm, 41 parts, among them J1 Conn_01x06, J2 PJ-102AH, J3 Conn_02x03_Odd_Even, SW1 Omron_B3F_SPST, SW2 Omron_B3F_SPST, SW3 Omron_B3F_SPST, SW4 Omron_B3F_SPST, U1 ATmega328-PU, U2 L7805, U3 MAX7219, U4 DS1307_DIP-8, Y1 Crystal_16MHz, Y2 Crystal_32768Hz

Commit message: ewwww
Parts:
- added J1: Conn_01x06, footprints:PinHeader_1x06_P2.54mm_Vertical, F.Cu at (96.5, 63.5)
- added J2: Power_inlet_vertical, footprints:Wurth-694106402002, F.Cu at (185.4, 68.6)
- added J4: Conn_01x03, footprints:PinHeader_1x03_P2.54mm_Vertical, F.Cu at (88.9, 76.2)
- added J5: Conn_01x03, footprints:PinHeader_1x03_P2.54mm_Vertical, F.Cu at (88.9, 94.0)
- moved U2 122.3 mm to (200.2, 133.1)
- moved J3 114.0 mm to (162.6, 132.1)
- moved J2 68.1 mm to (208.3, 76.2)
- moved R1 56.9 mm to (203.2, 94.0)
- moved Y2 54.4 mm to (203.2, 99.1)
- moved D1 54.0 mm to (203.2, 102.9)
- moved R9 45.7 mm to (202.3, 109.2)
- moved Y1 44.1 mm to (208.3, 88.9)
- moved J1 39.1 mm to (213.4, 102.9)
Connections:
- J3 pad 3: RESET -> LED_SCK
- J3 pad 5: LED_SCK -> RESET
- R2 pad 1: Net-(J1-Pad2) -> Net-(J1-Pad5)
- R2 pad 2: TXD -> RXD
- R3 pad 1: Net-(J1-Pad3) -> Net-(J1-Pad4)
- R3 pad 2: RXD -> TXD
- U1 pad 11: unconnected-(U1-Pad11) -> DEBUG_1
- U1 pad 12: unconnected-(U1-Pad12) -> DEBUG_2
- U1 pad 13: unconnected-(U1-Pad13) -> DEBUG_3
- U1 pad 24: unconnected-(U1-Pad24) -> DEBUG_4
- U1 pad 25: unconnected-(U1-Pad25) -> DEBUG_5
- U1 pad 26: unconnected-(U1-Pad26) -> DEBUG_6
- U3 pad 1: unconnected-(U3-Pad1) -> DISP_DATA
- U3 pad 12: unconnected-(U3-Pad12) -> DISP_LOAD
- U3 pad 13: unconnected-(U3-Pad13) -> DISP_CLK

Commit message: did a copper pour
Parts:
- removed the J1 at (213.4, 102.9)
- removed the J2 at (208.3, 76.2)
- J4, J5: value Conn_01x03 -> Conn_01x05; footprint footprints:PinHeader_1x03_P2.54mm_Vertical -> footprints:PinHeader_1x05_P2.54mm_Vertical
- moved SW1 224.6 mm to (93.6, 72.4)
- moved C2 221.3 mm to (94.0, 106.7), turned to 180 degrees
- moved R5 211.6 mm to (94.0, 124.5), turned to 180 degrees
- moved C1 209.9 mm to (94.0, 109.2), turned to 180 degrees
- moved R3 208.3 mm to (98.6, 85.1), turned to -90 degrees
- moved C9 187.5 mm to (149.9, 134.2), turned to -90 degrees
- moved R6 169.1 mm to (94.0, 127.0)
- moved R2 162.6 mm to (101.2, 85.1), turned to -90 degrees
- moved R4 161.4 mm to (90.2, 104.1), turned to 180 degrees
- moved C3 150.1 mm to (119.4, 101.6)
- moved C5 149.2 mm to (103.7, 74.9)
- moved R8 149.1 mm to (120.7, 94.0), turned to 180 degrees
- moved SW2 141.6 mm to (175.3, 134.6)
- moved R7 138.5 mm to (148.6, 128.7), turned to 90 degrees
- moved C8 135.3 mm to (152.4, 134.2), turned to -90 degrees
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Connections:
- J4 pad 1: DEBUG_4 -> VCC
- J4 pad 2: DEBUG_5 -> DEBUG_4
- J4 pad 3: DEBUG_6 -> DEBUG_5
- J5 pad 1: DEBUG_1 -> VCC
- J5 pad 2: DEBUG_2 -> DEBUG_1
- J5 pad 3: DEBUG_3 -> DEBUG_2

Commit message: lots o' changes
Parts:
- J2: moved to B.Cu
- moved J2 260.4 mm to (442.0, 125.3), turned to 180 degrees
- moved BT1 232.5 mm to (422.7, 90.6)
- moved C7 231.2 mm to (425.9, 129.1)
- moved C6 231.2 mm to (421.6, 122.3)
- moved U2 231.2 mm to (429.3, 124.0)
- moved U4 89.2 mm to (129.5, 131.7)
- moved Y2 88.7 mm to (133.3, 129.5)
- moved R4 77.3 mm to (156.2, 64.0), turned to 90 degrees
- moved J4 76.2 mm to (146.1, 64.0), turned to -90 degrees
- moved C4 72.1 mm to (184.2, 80.0)
- moved D1 72.1 mm to (156.2, 67.8), turned to -90 degrees
- moved C3 71.6 mm to (184.2, 71.1)
- moved Y1 71.6 mm to (179.1, 76.2)
- moved C2 71.2 mm to (153.7, 67.8), turned to 90 degrees
- moved C1 70.6 mm to (151.1, 67.8), turned to 90 degrees
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- renumbered H4 to locked, H2 to locked, H3 to locked, H1 to locked
Connections:
- J5 pad 1: VCC -> DEBUG_1
- J5 pad 2: DEBUG_1 -> DEBUG_2
- J5 pad 3: DEBUG_2 -> DEBUG_3
- J5 pad 4: DEBUG_3 -> VCC
- R6 pad 2: SCL -> SDA
- U1 pad 27: SCL -> SDA
- U4 pad 5: SCL -> SDA
Routing:
- added copper zone on B.Cu, net GND
- added copper zone on F.Cu, net VCC

Commit message: new traces
Parts:
- moved J2 350.6 mm to (91.4, 120.7), turned to 90 degrees
- moved C6 334.1 mm to (87.6, 129.1)
- moved C7 334.1 mm to (91.9, 135.9)
- moved U2 334.1 mm to (95.2, 130.8)
- moved BT1 326.6 mm to (96.5, 106.9), turned to 90 degrees
- moved C4 40.1 mm to (144.8, 87.6), turned to 180 degrees
- moved Y1 28.3 mm to (153.2, 87.6), turned to 180 degrees
- moved C3 27.2 mm to (162.6, 87.6)
- moved R9 10.2 mm to (113.0, 87.6), turned to 180 degrees
- moved R5 3.59 mm to (116.8, 125.7)
- moved R6 3.59 mm to (116.8, 123.2)
- moved R8 3.06 mm to (113.9, 94.0), turned to 90 degrees
- moved U4 0.85 mm to (129.5, 130.8)
Routing:
- net Net-(DS1-Pad3): track 0.00 -> 138.3 mm
- net Net-(DS1-Pad5): track 0.00 -> 84.0 mm
- net SCL: track 0.00 -> 77.7 mm
- net MOSI: track 0.00 -> 70.7 mm
- net MISO: track 0.00 -> 66.1 mm
- net Net-(DS1-Pad13): track 0.00 -> 65.7 mm
- net SDA: track 0.00 -> 61.6 mm
- net LED_SCK: track 0.00 -> 60.9 mm
- net Net-(DS1-Pad11): track 0.00 -> 59.9 mm
- net Net-(DS1-Pad12): track 0.00 -> 59.5 mm
- net GND: track 0.00 -> 56.4 mm, vias 0 -> 4
- net Net-(DS1-Pad10): track 0.00 -> 54.8 mm
- net Net-(DS1-Pad9): track 0.00 -> 49.4 mm
- net Net-(BT1-Pad1): track 0.00 -> 45.7 mm
- net Net-(DS1-Pad14): track 0.00 -> 44.6 mm
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
Commit message: pretty close to done
Parts:
- moved R10 25.4 mm to (198.1, 129.5)
- moved R12 25.4 mm to (172.7, 129.5), turned to 90 degrees
- moved SW2 25.4 mm to (191.8, 126.2)
- moved SW4 25.4 mm to (166.4, 126.2)
Connections:
- U1 pad 4: BTH_DWN -> BTN_DWN
Routing:
- net DISP_DATA: track 0.00 -> 131.2 mm
- net Net-(DS1-Pad1): track 0.00 -> 123.6 mm
- net BTN_UP: track 0.00 -> 113.4 mm
- net BTN_SEL: track 0.00 -> 98.1 mm
- net BTN_DWN: track 0.00 -> 83.4 mm
- net DISP_CLK: track 0.00 -> 81.2 mm
- net Net-(DS1-Pad2): track 0.00 -> 66.9 mm
- net Net-(DS1-Pad4): track 0.00 -> 66.4 mm
- net LIGHT_SENSOR: track 2.95 -> 45.9 mm
- net TXD: track 0.00 -> 39.6 mm, vias 0 -> 1
- net RXD: track 0.00 -> 34.2 mm, vias 0 -> 1
- net RESET: track 12.2 -> 45.0 mm

Commit message: 70% there
Parts:
- moved J4 2.55 mm to (143.5, 64.0)
Connections:
- J4 pad 1: VCC -> DEBUG_4
- J4 pad 2: DEBUG_4 -> DEBUG_5
- J4 pad 3: DEBUG_5 -> DEBUG_6
- J4 pad 4: DEBUG_6 -> VCC
Routing:
- net DISP_LOAD: track 0.00 -> 63.4 mm
- net GND: track 56.4 -> 88.0 mm, vias 4 -> 7
Changed lines of the file:
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@@
   )
   (footprint "footprints:PinHeader_1x05_P2.54mm_Vertical" (layer "F.Cu")
-    (at 146.05 63.97 -90)
+    (at 143.505 63.97 -90)
     (descr "Through hole straight pin header, 1x05, 2.54mm pitch, single row")
     (tags "Through hole pin header THT 1x05 2.54mm single row")
@@
     (fp_line (start 1.27 -1.27) (end 1.27 11.43) (layer "F.Fab") (width 0.1))
     (pad "1" thru_hole rect locked (at 0 0 270) (size 1.7 1.7) (drill 1) (layers *.Cu *.Mask)
-      (net 4 "VCC") (pinfunction "Pin_1") (pintype "passive"))
+      (net 41 "DEBUG_4") (pinfunction "Pin_1") (pintype "passive"))
     (pad "2" thru_hole oval locked (at 0 2.54 270) (size 1.7 1.7) (drill 1) (layers *.Cu *.Mask)
-      (net 41 "DEBUG_4") (pinfunction "Pin_2") (pintype "passive"))
+      (net 42 "DEBUG_5") (pinfunction "Pin_2") (pintype "passive"))
     (pad "3" thru_hole oval locked (at 0 5.08 270) (size 1.7 1.7) (drill 1) (layers *.Cu *.Mask)
-      (net 42 "DEBUG_5") (pinfunction "Pin_3") (pintype "passive"))
+      (net 43 "DEBUG_6") (pinfunction "Pin_3") (pintype "passive"))
     (pad "4" thru_hole oval locked (at 0 7.62 270) (size 1.7 1.7) (drill 1) (layers *.Cu *.Mask)
-      (net 43 "DEBUG_6") (pinfunction "Pin_4") (pintype "passive"))
+      (net 4 "VCC") (pinfunction "Pin_4") (pintype "passive"))
     (pad "5" thru_hole oval locked (at 0 10.16 270) (size 1.7 1.7) (drill 1) (layers *.Cu *.Mask)
       (net 2 "GND") (pinfunction "Pin_5") (pintype "passive"))
@@
   (segment (start 96.520017 111.064074) (end 114.131863 128.67592) (width 0.2032) (layer "F.Cu") (net 1))
   (segment (start 96.520017 106.863686) (end 96.520017 111.064074) (width 0.2032) (layer "F.Cu") (net 1))
+  (segment (start 147.32 82.55) (end 143.93 85.94) (width 0.2032) (layer "F.Cu") (net 2))
+  (segment (start 143.93 87.63) (end 140.97 87.63) (width 0.2032) (layer "F.Cu") (net 2))
   (segment (start 118.11 69.05) (end 118.11 67.31) (width 0.2032) (layer "F.Cu") (net 2))
   (segment (start 97.35 131.25) (end 97.35 130.81) (width 0.508) (layer "F.Cu") (net 2))
+  (segment (start 151.14 79.2) (end 151.14 81.27) (width 0.2032) (layer "F.Cu") (net 2))
   (segment (start 97.79 125.73) (end 99.06 125.73) (width 0.508) (layer "F.Cu") (net 2))
   (segment (start 87.63 129.97) (end 87.63 130.81) (width 0.508) (layer "F.Cu") (net 2))
@@
   (segment (start 96.51 129.97) (end 97.35 130.81) (width 0.508) (layer "F.Cu") (net 2))
   (segment (start 92.71 135.89) (end 97.35 131.25) (width 0.508) (layer "F.Cu") (net 2))
+  (segment (start 143.93 85.94) (end 143.93 87.63) (width 0.2032) (layer "F.Cu") (net 2))
   (segment (start 87.63 130.81) (end 86.36 132.08) (width 0.508) (layer "F.Cu") (net 2))
+  (segment (start 163.41 87.63) (end 164.305 87.63) (width 0.2032) (layer "F.Cu") (net 2))
   (segment (start 121.92 63.97) (end 119.85 66.04) (width 0.2032) (layer "F.Cu") (net 2))
+  (segment (start 149.86 82.55) (end 147.32 82.55) (width 0.2032) (layer "F.Cu") (net 2))
   (segment (start 86.14 121.85) (end 95.18 121.85) (width 0.508) (layer "F.Cu") (net 2))
+  (segment (start 168.915 83.02) (end 173.52 83.02) (width 0.2032) (layer "F.Cu") (net 2))
   (segment (start 97.35 124.02) (end 97.35 125.29) (width 0.508) (layer "F.Cu") (net 2))
   (segment (start 119.38 66.04) (end 119.38 63.97) (width 0.2032) (layer "F.Cu") (net 2))
+  (segment (start 151.14 81.27) (end 149.86 82.55) (width 0.2032) (layer "F.Cu") (net 2))
   (segment (start 92.71 137.16) (end 93.98 138.43) (width 0.508) (layer "F.Cu") (net 2))
+  (segment (start 195.58 88.9) (end 196.85 87.63) (width 0.2032) (layer "F.Cu") (net 2))
   (segment (start 92.71 135.89) (end 92.71 137.16) (width 0.508) (layer "F.Cu") (net 2))
   (segment (start 191.77 88.9) (end 194.31 88.9) (width 0.2032) (layer "F.Cu") (net 2))
   (segment (start 95.18 121.85) (end 97.35 124.02) (width 0.508) (layer "F.Cu") (net 2))
+  (segment (start 164.305 87.63) (end 168.915 83.02) (width 0.2032) (layer "F.Cu") (net 2))
   (segment (start 87.63 129.97) (end 96.51 129.97) (width 0.508) (layer "F.Cu") (net 2))
   (segment (start 97.35 125.29) (end 97.35 130.81) (width 0.508) (layer "F.Cu") (net 2))
+  (segment (start 173.52 83.02) (end 173.99 82.55) (width 0.2032) (layer "F.Cu") (net 2))
   (segment (start 97.35 125.29) (end 97.79 125.73) (width 0.508) (layer "F.Cu") (net 2))
+  (segment (start 194.31 88.9) (end 195.58 88.9) (width 0.2032) (layer "F.Cu") (net 2))
+  (via (at 173.99 82.55) (size 0.8128) (drill 0.4064) (layers "F.Cu" "B.Cu") (net 2))
+  (via (at 140.97 87.63) (size 0.8128) (drill 0.4064) (layers "F.Cu" "B.Cu") (net 2))
   (via (at 118.11 66.04) (size 0.8128) (drill 0.4064) (layers "F.Cu" "B.Cu") (net 2))
   (via (at 99.06 125.73) (size 0.8128) (drill 0.4064) (layers "F.Cu" "B.Cu") (net 2))
   (via (at 86.36 132.08) (size 0.8128) (drill 0.4064) (layers "F.Cu" "B.Cu") (net 2))
+  (via (at 196.85 87.63) (size 0.8128) (drill 0.4064) (layers "F.Cu" "B.Cu") (net 2))
   (via (at 93.98 138.43) (size 0.8128) (drill 0.4064) (layers "F.Cu" "B.Cu") (net 2))
   (segment (start 151.13 71.57) (end 151.14 71.58) (width 0.2032) (layer "F.Cu") (net 3))
@@
   (segment (start 138.43 63.97) (end 138.43 71.57) (width 0.2032) (layer "F.Cu") (net 43))
   (segment (start 138.43 71.57) (end 138.44 71.58) (width 0.2032) (layer "F.Cu") (net 43))
+  (segment (start 208.28 96.52) (end 208.28 104.125) (width 0.2032) (layer "B.Cu") (net 44))
+  (segment (start 166.38 79.2) (end 167.64 80.46) (width 0.2032) (layer "B.Cu") (net 44))
+  (segment (start 167.64 80.46) (end 167.64 88.9) (width 0.2032) (layer "B.Cu") (net 44))
+  (segment (start 207.46816 95.70816) (end 208.28 96.52) (width 0.2032) (layer "B.Cu") (net 44))
+  (segment (start 208.28 104.125) (end 207.005 105.4) (width 0.2032) (layer "B.Cu") (net 44))
+  (segment (start 167.64 88.9) (end 174.44816 95.70816) (width 0.2032) (layer "B.Cu") (net 44))
+  (segment (start 174.44816 95.70816) (end 207.46816 95.70816) (width 0.2032) (layer "B.Cu") (net 44))
   (segment (start 158.755 83.02) (end 158.755 79.205) (width 0.2032) (layer "F.Cu") (net 45))
   (segment (start 158.755 79.205) (end 158.76 79.2) (width 0.2032) (layer "F.Cu") (net 45))

Commit message: pre check finish
Parts:
- moved SW2 0.42 mm to (191.8, 125.7)
Routing:
- net Net-(DS1-Pad3): track 138.3 -> 48.7 mm
- net Net-(DS1-Pad1): track 123.6 -> 50.0 mm, vias 0 -> 4
- net Net-(DS1-Pad11): track 59.9 -> 93.6 mm, vias 0 -> 3
- net GND: track 88.0 -> 119.8 mm, vias 7 -> 14
- net Net-(DS1-Pad5): track 84.0 -> 56.3 mm
- net DISP_CLK: track 81.2 -> 53.7 mm
- net Net-(DS1-Pad2): track 66.9 -> 41.0 mm
- net DISP_DATA: track 131.2 -> 105.3 mm, vias 0 -> 2
- net Net-(DS1-Pad4): track 66.4 -> 43.6 mm
- net RESET: track 45.0 -> 61.9 mm, vias 0 -> 3
- net Net-(DS1-Pad12): track 59.5 -> 66.6 mm, vias 0 -> 2
- net Net-(DS1-Pad10): track 54.8 -> 47.8 mm, vias 0 -> 2
- net DISP_LOAD: track 63.4 -> 57.8 mm
- net Net-(DS1-Pad13): track 65.7 -> 70.0 mm
- net Net-(DS1-Pad14): track 44.6 -> 48.3 mm, vias 0 -> 2
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
Commit message: DRC Checked!
Parts:
- moved C4 1.27 mm to (143.5, 87.6)
Routing:
- net GND: track 119.8 -> 118.6 mm
- net MISO: track 66.1 -> 64.8 mm
- net Net-(C4-Pad1): track 13.7 -> 15.0 mm
- net Net-(DS1-Pad1): track 50.0 -> 48.8 mm, vias 4 -> 2
